Commit message: some updates

File: gym_flexassembly/data/kuka-iiwa-7-egp-40/model.urdf (robot description, URDF)
Before this commit: robot kuka-iiwa-7-egp-40, 12 links, 11 joints
Links:
- removed link SchunkEGP40_link
- added link iiwa7_link_ee, mass 0.6; collision mesh filename=model://schunk-egp-40/meshes/visual/dae/schunk-egp-40-colli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 scale=1 1 1; visual mesh filename=model://schunk-egp-40/meshes/visual/obj/schunk_low_baked_sm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 scale=1 1 1
Joints:
- joint SchunkEGP40_Finger1_joint: parent SchunkEGP40_link -> iiwa7_link_ee
- joint SchunkEGP40_Finger2_joint: parent SchunkEGP40_link -> iiwa7_link_ee
- joint iiwa7_joint_ee: child SchunkEGP40_link -> iiwa7_link_ee
