Commit message: added description for the ati gamma

File: gym_flexassembly/data/robots/epfl-iiwa14/iiwa14.urdf (robot description, URDF)
Before this commit: robot iiwa14, 12 links, 11 joints
Links:
- added link ft_sensor, mass 0.215; collision mesh filename=model://ati-gamma/meshes/ati_gamma.stl; visual mesh filename=model://ati-gamma/meshes/ati_gamma.stl
Joints:
- added joint iiwa7_joint_ft_sensor: type fixed, parent iiwa_link_7, child ft_sensor, origin xyz=0 0 0.059 rpy=0 0 0
- joint iiwa7_joint_ee: origin xyz=0 0 0.126 rpy=0 0 0 -> xyz=0 0 0.01 rpy=0 0 0; parent iiwa_link_7 -> ft_sensor
